Commit message: started working on urdf file

File: jopdorp_robot_urdf.urdf (robot description, URDF)
Before this commit: robot materials, 9 links, 8 joints
Links:
- removed link base
- added link base_link; visual box size=0.6 0.1 0.2
Joints:
- joint shoulder_rotate: parent base -> base_link
- joint stretch_elbow_from_shoulder: child elbow_control -> elbow_control_link

Commit message: edded lengths to robot parts and joint positions

File: jopdorp_robot_urdf.urdf (robot description, URDF)
Before this commit: robot jopdorp_robot, 9 links, 8 joints
Links:
- removed link elbow_control_link
- removed link upper_arm_parallel
- link base_link: geometry visual box size=1 0.5 0.2
- link elbow_block: geometry visual box size=0.4 0.4 0.2
- link hand: geometry visual box size=0.2 0.3 0.05
- link lower_arm: geometry visual box size=0.1 1 0.1
- link shoulder_block: geometry visual box size=0.5 0.7 0.3
- link upper_arm: geometry visual box size=0.4 1 0.1
- link wrist_block: geometry visual box size=0.3 0.3 0.1
Joints:
- removed joint elbow_stretch_corner_joint
- removed joint stretch_elbow
- removed joint stretch_elbow_from_shoulder
- added joint inner_elbow: type fixed, parent upper_arm, child elbow_block, origin xyz=0 -1 0.2
- joint close_hand: origin xyz=0 0.22 0.25 -> xyz=0 0.2 0
- joint rotate_elbow: origin xyz=0 0.22 0.25 -> xyz=0 0.4 0
- joint shoulder_rotate: origin xyz=0 -0.22 0.25 -> xyz=0 0 0.3
- joint shoulder_stretch: origin xyz=0 -0.22 0.25 -> xyz=0 0.3 0
- joint wrist: origin xyz=0 0.22 0.25 -> xyz=0 0.5 0
